File: sendit/sendit.kicad_sch (KiCad schematic)
At the start: 7 parts, among them U1 ADS1115IDGS

Commit message: updated schematic.
Parts:
- removed C1: 100nF, Capacitor_SMD:C_0805_2012Metric_Pad1.18x1.45mm_HandSolder, symbol Device:C_Small
- removed C2: 10uF, Capacitor_SMD:C_0805_2012Metric_Pad1.18x1.45mm_HandSolder, symbol Device:C_Small
- removed D1: BAT54S, Package_TO_SOT_SMD:SOT-23, symbol Diode:BAT54S
- removed INPUT1: Conn_01x03, Connector_Phoenix_MC:PhoenixContact_MC_1,5_3-G-3.5_1x03_P3.50mm_Horizontal, symbol Connector_Generic:Conn_01x03
- removed R1: 249 0.1%, Resistor_SMD:R_1206_3216Metric_Pad1.30x1.75mm_HandSolder, symbol Device:R_Small_US
- removed R2: 10k, Resistor_SMD:R_0805_2012Metric_Pad1.20x1.40mm_HandSolder, symbol Device:R_Small_US
- removed U1: ADS1115IDGS, Package_SO:TSSOP-10_3x3mm_P0.5mm, symbol Analog_ADC:ADS1015IDGS
- added U2: Seeed_Studio_XIAO_ESP32C6, Seeed Studio XIAO Series Library:XIAO-Generic-Hybrid-14P-2.54-21X17.8MM, symbol yarrboard:Seeed_Studio_XIAO_ESP32C6
Connections:
- net +5V: now also U2.14 (5V)
- net SCL: now also U2.6 (D5)
- net SDA: now also U2.5 (D4)
- new net GND: U2.13 (GND)
Other:
- added sheet ADC1 (1115_adc.kicad_sch)
- added sheet ADC2 (1115_adc.kicad_sch)
- added sheet SENDER 1 (sender.kicad_sch)
- added sheet SENDER 2 (sender.kicad_sch)
- added sheet SENDER 3 (sender.kicad_sch)
- added sheet SENDER 4 (sender.kicad_sch)
- added sheet SENDER 5 (sender.kicad_sch)
- added sheet SENDER 6 (sender.kicad_sch)
- added sheet SENDER 7 (sender.kicad_sch)
- added sheet SENDER 8 (sender.kicad_sch)
